File: KiCad/WilliamsAlarm.sch (KiCad schematic (older format))
At the start: 27 parts

Commit message: update resistor names
Parts:
- gave numbers to parts that had none: 14
Changed lines of the file:
@@
 	2350 3000 3650 3000
 $Comp
-L Device:R_US R?
+L Device:R_US R3
 U 1 1 5B96C406
 P 3900 1150
-F 0 "R?" H 3968 1196 50  0000 L CNN
+F 0 "R3" H 3968 1196 50  0000 L CNN
 F 1 "3k3" H 3968 1105 50  0000 L CNN
 F 2 "" V 3940 1140 50  0001 C CNN
@@
 $EndComp
 $Comp
-L Device:R_US R?
+L Device:R_US R5
 U 1 1 5B96C42C
 P 4150 1150
-F 0 "R?" H 4218 1196 50  0000 L CNN
+F 0 "R5" H 4218 1196 50  0000 L CNN
 F 1 "3k3" H 4218 1105 50  0000 L CNN
 F 2 "" V 4190 1140 50  0001 C CNN
@@
 $EndComp
 $Comp
-L Device:R_US R?
+L Device:R_US R7
 U 1 1 5B96C459
 P 4400 1150
-F 0 "R?" H 4468 1196 50  0000 L CNN
+F 0 "R7" H 4468 1196 50  0000 L CNN
 F 1 "3k3" H 4468 1105 50  0000 L CNN
 F 2 "" V 4440 1140 50  0001 C CNN
@@
 $EndComp
 $Comp
-L Device:R_US R?
+L Device:R_US R9
 U 1 1 5B96C489
 P 4650 1150
-F 0 "R?" H 4718 1196 50  0000 L CNN
+F 0 "R9" H 4718 1196 50  0000 L CNN
 F 1 "3k3" H 4718 1105 50  0000 L CNN
 F 2 "" V 4690 1140 50  0001 C CNN
@@
 $EndComp
 $Comp
-L Device:R_US R?
+L Device:R_US R11
 U 1 1 5B96C502
 P 4900 1150
-F 0 "R?" H 4968 1196 50  0000 L CNN
+F 0 "R11" H 4968 1196 50  0000 L CNN
 F 1 "3k3" H 4968 1105 50  0000 L CNN
 F 2 "" V 4940 1140 50  0001 C CNN
@@
 $EndComp
 $Comp
-L Device:R_US R?
+L Device:R_US R13
 U 1 1 5B96C52C
 P 5150 1150
-F 0 "R?" H 5218 1196 50  0000 L CNN
+F 0 "R13" H 5218 1196 50  0000 L CNN
 F 1 "3k3" H 5218 1105 50  0000 L CNN
 F 2 "" V 5190 1140 50  0001 C CNN
@@
 $EndComp
 $Comp
-L Device:R_US R?
+L Device:R_US R15
 U 1 1 5B96C560
 P 5400 1150
-F 0 "R?" H 5468 1196 50  0000 L CNN
+F 0 "R15" H 5468 1196 50  0000 L CNN
 F 1 "3k3" H 5468 1105 50  0000 L CNN
 F 2 "" V 5440 1140 50  0001 C CNN
@@
 $EndComp
 $Comp
-L Device:R_US R?
+L Device:R_US R4
 U 1 1 5B96C624
 P 3900 2850
-F 0 "R?" H 3832 2804 50  0000 R CNN
+F 0 "R4" H 3832 2804 50  0000 R CNN
 F 1 "3k3" H 3832 2895 50  0000 R CNN
 F 2 "" V 3940 2840 50  0001 C CNN
@@
 $EndComp
 $Comp
-L Device:R_US R?
+L Device:R_US R6
 U 1 1 5B96C660
 P 4150 2850
-F 0 "R?" H 4082 2804 50  0000 R CNN
+F 0 "R6" H 4082 2804 50  0000 R CNN
 F 1 "3k3" H 4082 2895 50  0000 R CNN
 F 2 "" V 4190 2840 50  0001 C CNN
@@
 $EndComp
 $Comp
-L Device:R_US R?
+L Device:R_US R8
 U 1 1 5B96C6AA
 P 4400 2850
-F 0 "R?" H 4332 2804 50  0000 R CNN
+F 0 "R8" H 4332 2804 50  0000 R CNN
 F 1 "3k3" H 4332 2895 50  0000 R CNN
 F 2 "" V 4440 2840 50  0001 C CNN
@@
 $EndComp
 $Comp
-L Device:R_US R?
+L Device:R_US R10
 U 1 1 5B96C6DA
 P 4650 2850
-F 0 "R?" H 4582 2804 50  0000 R CNN
+F 0 "R10" H 4582 2804 50  0000 R CNN
 F 1 "3k3" H 4582 2895 50  0000 R CNN
 F 2 "" V 4690 2840 50  0001 C CNN
@@
 $EndComp
 $Comp
-L Device:R_US R?
+L Device:R_US R12
 U 1 1 5B96C70C
 P 4900 2850
-F 0 "R?" H 4832 2804 50  0000 R CNN
+F 0 "R12" H 4832 2804 50  0000 R CNN
 F 1 "3k3" H 4832 2895 50  0000 R CNN
 F 2 "" V 4940 2840 50  0001 C CNN
@@
 $EndComp
 $Comp
-L Device:R_US R?
+L Device:R_US R14
 U 1 1 5B96C744
 P 5150 2850
-F 0 "R?" H 5082 2804 50  0000 R CNN
+F 0 "R14" H 5082 2804 50  0000 R CNN
 F 1 "3k3" H 5082 2895 50  0000 R CNN
 F 2 "" V 5190 2840 50  0001 C CNN
@@
 	5150 1300 5150 1350
 $Comp
-L Device:R_US R?
+L Device:R_US R16
 U 1 1 5B96CD3A
 P 5400 2850
-F 0 "R?" H 5332 2804 50  0000 R CNN
+F 0 "R16" H 5332 2804 50  0000 R CNN
 F 1 "3k3" H 5332 2895 50  0000 R CNN
 F 2 "" V 5440 2840 50  0001 C CNN

Commit message: add status LED's
Parts:
- added D1, D10, D2, D3, D4, D5, D6, D7, D9: LED, symbol Device:LED
- added R17, R18, R19, R20, R21, R22, R23, R24, R25: 330, symbol Device:R_US
- added SW1, SW2: (no value), symbol Switch:SW_Push
- gave numbers to parts that had none: 2
- renumbered D1 to D8
Connections:
- wire segments 60 -> 96
Other:
- note added: "Arm"
- note added: "Arm/Disarm"
- note added: "LED Status panel"
- note added: "Panic"
- note added: "Ready"
- note added: "Z1"
- note added: "Z2"
- note added: "Z3"
- note added: "Z4"
- note added: "Z5"
- note added: "Z6"
- note added: "Z7"
- note added: "Z8"

Commit message: add alarm output
Parts:
- added D9: LED, symbol Device:LED
- added R?: 330, symbol Device:R_US
- renumbered D9 to D10, D10 to D11
Connections:
- wire segments 96 -> 99
Other:
- note added: "Alarm"
Changed lines of the file:
@@
-$EndComp
-$Comp
-L Device:R_US R15
-U 1 1 5B96C560
-P 8550 2550
-F 0 "R15" H 8618 2596 50  0000 L CNN
-F 1 "3k3" H 8618 2505 50  0000 L CNN
-F 2 "" V 8590 2540 50  0001 C CNN
-F 3 "~" H 8550 2550 50  0001 C CNN
-	1    8550 2550
-	1    0    0    -1
 $EndComp
 $Comp
@@
 Wire Wire Line
 	8300 2700 8300 2750
-$Comp
-L Device:R_US R16
-U 1 1 5B96CD3A
-P 8550 4500
-F 0 "R16" H 8482 4454 50  0000 R CNN
-F 1 "3k3" H 8482 4545 50  0000 R CNN
-F 2 "" V 8590 4490 50  0001 C CNN
-F 3 "~" H 8550 4500 50  0001 C CNN
-	1    8550 4500
-	-1   0    0    1
-$EndComp
 Wire Wire Line
 	8550 2700 8550 2750
@@
 Connection ~ 8050 3750
 Connection ~ 8300 3850
-Connection ~ 8550 3950
 Wire Wire Line
 	6800 4650 7050 4650
@@
 Connection ~ 8050 4650
 Wire Wire Line
-	8300 4650 8550 4650
-Connection ~ 8300 4650
-Wire Wire Line
 	7050 2050 6800 2050
 Connection ~ 6800 2050
@@
 	8300 2050 8050 2050
 Connection ~ 8050 2050
-Wire Wire Line
-	8550 2050 8300 2050
-Connection ~ 8300 2050
 $Comp
 L Device:R_US R26
@@
 Wire Wire Line
 	8300 3150 8300 3850
-Wire Wire Line
-	8550 3150 8550 3950
 $Comp
 L Switch:SW_Reed_Opener Z1
@@
 $EndComp
 $Comp
-L Switch:SW_Reed_Opener Z8
-U 1 1 5B974E55
-P 8550 2950
-F 0 "Z8" V 8504 3035 50  0000 L CNN
-F 1 " " V 8595 3035 50  0000 L CNN
-F 2 "" H 8550 2950 50  0001 C CNN
-F 3 "" H 8550 2950 50  0001 C CNN
-	1    8550 2950
-	0    1    1    0
-$EndComp
-$Comp
 L Device:R_US R25
 U 1 1 5B983241
@@
 	8300 3850 8300 4350
 Wire Wire Line
-	8550 3950 8550 4350
-Wire Wire Line
 	5000 4050 5000 3950
 Wire Wire Line
@@
 Connection ~ 2900 4650
 $Comp
-L Device:LED D10
+L Device:LED D11
 U 1 1 5B9AA785
 P 2600 4200
-F 0 "D10" H 2591 4416 50  0000 C CNN
+F 0 "D11" H 2591 4416 50  0000 C CNN
 F 1 "LED" H 2591 4325 50  0000 C CNN
 F 2 "" H 2600 4200 50  0001 C CNN
@@
 $EndComp
 $Comp
-L Device:LED D9
+L Device:LED D10
 U 1 1 5B9AA7F9
 P 2300 4200
-F 0 "D9" H 2291 4416 50  0000 C CNN
+F 0 "D10" H 2291 4416 50  0000 C CNN
 F 1 "LED" H 2291 4325 50  0000 C CNN
 F 2 "" H 2300 4200 50  0001 C CNN
@@
 	8300 2050 8300 2400
 Wire Wire Line
-	8550 2050 8550 2400
-Wire Wire Line
 	6100 2050 6100 2250
 Text Notes 6750 4800 0    50   ~ 0
@@
 Text Notes 8250 4800 0    50   ~ 0
 Z7
-Text Notes 8500 4800 0    50   ~ 0
-Z8
 $Comp
 L Switch:SW_Push SW2
@@
 	4950 2050 4950 2150
 Connection ~ 6100 2050
-Wire Wire Line
-	4950 2550 4950 2850
-Wire Wire Line
-	4950 2850 5400 2850
 Text Notes 5000 2250 0    50   ~ 0
 Arm/Disarm
@@
 Wire Wire Line
 	6400 3850 8300 3850
-Wire Wire Line
-	6400 3950 8550 3950
 Wire Wire Line
 	6000 4650 6800 4650
@@
 	5000 4650 6000 4650
 Connection ~ 4950 2050
-Wire Wire Line
-	4450 2550 4450 2950
-Wire Wire Line
-	4450 2950 5400 2950
 Text Notes 4500 2250 0    50   ~ 0
 Panic
 Text Notes 3350 4950 0    50   ~ 0
 LED Status panel
+Text Notes 8500 4800 0    50   ~ 0
+Z8
+Wire Wire Line
+	8550 2050 8550 2400
+Connection ~ 8300 2050
+Wire Wire Line
+	8550 2050 8300 2050
+$Comp
+L Device:R_US R15
+U 1 1 5B96C560
+P 8550 2550
+F 0 "R15" H 8618 2596 50  0000 L CNN
+F 1 "3k3" H 8618 2505 50  0000 L CNN
+F 2 "" V 8590 2540 50  0001 C CNN
+F 3 "~" H 8550 2550 50  0001 C CNN
+	1    8550 2550
+	1    0    0    -1
+$EndComp
+$Comp
+L Switch:SW_Reed_Opener Z8
+U 1 1 5B974E55
+P 8550 2950
+F 0 "Z8" V 8504 3035 50  0000 L CNN
+F 1 " " V 8595 3035 50  0000 L CNN
+F 2 "" H 8550 2950 50  0001 C CNN
+F 3 "" H 8550 2950 50  0001 C CNN
+	1    8550 2950
+	0    1    1    0
+$EndComp
+Connection ~ 8300 4650
+Wire Wire Line
+	8300 4650 8550 4650
+$Comp
+L Device:R_US R16
+U 1 1 5B96CD3A
+P 8550 4500
+F 0 "R16" H 8482 4454 50  0000 R CNN
+F 1 "3k3" H 8482 4545 50  0000 R CNN
+F 2 "" V 8590 4490 50  0001 C CNN
+F 3 "~" H 8550 4500 50  0001 C CNN
+	1    8550 4500
+	-1   0    0    1
+$EndComp
+Wire Wire Line
+	8550 3950 8550 4350
+Wire Wire Line
+	8550 3150 8550 3950
+Connection ~ 8550 3950
+Wire Wire Line
+	6400 3950 8550 3950
+$Comp
+L Device:R_US R?
+U 1 1 5B99AD78
+P 2000 4500
+F 0 "R?" H 1932 4454 50  0000 R CNN
+F 1 "330" H 1932 4545 50  0000 R CNN
+F 2 "" V 2040 4490 50  0001 C CNN
+F 3 "~" H 2000 4500 50  0001 C CNN
+	1    2000 4500
+	-1   0    0    1
+$EndComp
+$Comp
+L Device:LED D9
+U 1 1 5B99ADF8
+P 2000 4200
+F 0 "D9" H 1991 4416 50  0000 C CNN
+F 1 "LED" H 1991 4325 50  0000 C CNN
+F 2 "" H 2000 4200 50  0001 C CNN
+F 3 "~" H 2000 4200 50  0001 C CNN
+	1    2000 4200
+	0    -1   -1   0
+$EndComp
+Wire Wire Line
+	2000 4650 2300 4650
+Connection ~ 2300 4650
+Wire Wire Line
+	5400 2950 2000 2950
+Wire Wire Line
+	2000 2950 2000 4050
+Wire Wire Line
+	4950 2650 5400 2650
+Wire Wire Line
+	4950 2550 4950 2650
+Wire Wire Line
+	4450 2550 4450 2750
+Wire Wire Line
+	4450 2750 5400 2750
+Text Notes 1900 4800 0    50   ~ 0
+Alarm
 $EndSCHEMATC
